File: stm32_bluepill/stm32_bluepill.kicad_sch (KiCad schematic)
At the start: 29 parts, among them J1 USB_B_Micro, J2 Conn_01x04_Pin, J4 Conn_01x04_Pin, J5 Conn_01x04_Pin, J6 Conn_01x08_Pin, SW1 SW_SPDT, U1 STM32F103C8T6, U2 AMS1117-3.3, Y1 16MHz

Commit message: PCB components located
Parts:
- added H1, H2, H3, H4: MountingHole, MountingHole:MountingHole_2.2mm_M2, symbol Mechanical:MountingHole
- added J3: Conn_01x01_MountingPin, symbol Connector_Generic_MountingPin:Conn_01x01_MountingPin
- C1, C10, C11, C2, C3, C4, C6, C7, C8, C9: footprint (none) -> Capacitor_SMD:C_0402_1005Metric
- C12, C13: value 1u -> 22u; footprint (none) -> Capacitor_SMD:C_0805_2012Metric
- C5: footprint (none) -> Capacitor_SMD:C_0603_1608Metric
- D1: footprint (none) -> LED_SMD:LED_0603_1608Metric
- FB1: footprint (none) -> Inductor_SMD:L_0603_1608Metric
- J1: footprint (none) -> Connector_USB:USB_Micro-B_Wuerth_629105150521
- J2, J4, J5: footprint (none) -> Connector_PinHeader_2.54mm:PinHeader_1x04_P2.54mm_Vertical
- J6: footprint (none) -> Connector_PinHeader_2.54mm:PinHeader_1x08_P2.54mm_Vertical
- R1, R2, R3, R4, R5: footprint (none) -> Resistor_SMD:R_0402_1005Metric
- SW1: footprint (none) -> Button_Switch_SMD:SW_SPDT_PCM12
- Y1: footprint (none) -> Crystal:Crystal_SMD_3225-4Pin_3.2x2.5mm_HandSoldering

Commit message: Add files via upload
Parts:
- removed J3: Conn_01x01_MountingPin, symbol Connector_Generic_MountingPin:Conn_01x01_MountingPin
- removed SW1: SW_SPDT, Button_Switch_SMD:SW_SPDT_PCM12, symbol Switch:SW_SPDT
- added J7: Conn_01x03_Pin, Connector_PinHeader_2.54mm:PinHeader_1x03_P2.54mm_Vertical, symbol Connector:Conn_01x03_Pin
Connections:
- net +3.3V: now also J7.1 (Pin_1)
- net GND: now also J7.3 (Pin_3)
- net SW_BOOT0: now also J7.2 (Pin_2)
